File: TPS922055 Module.kicad_sch (KiCad schematic)
At the start: 26 parts, among them J1 Conn_01x04_Pin, J2 Conn_01x04_Pin, J3 Conn_01x02_Pin, U1 TPS922055DRRR

Commit message: Refinements, Increased module size to fit heatsink better
Parts:
- removed J1: Conn_01x04_Pin, Connector_PinSocket_2.54mm:PinSocket_1x04_P2.54mm_Vertical, symbol Connector:Conn_01x04_Pin
- removed J3: Conn_01x02_Pin, Connector_PinSocket_2.54mm:PinSocket_1x02_P2.54mm_Vertical, symbol Connector:Conn_01x02_Pin
- added C41: 10uF, Capacitor_SMD:C_1210_3225Metric, symbol Device:C_Small
- added J1: Conn_01x07_Socket, Connector_PinSocket_2.54mm:PinSocket_1x07_P2.54mm_Vertical, symbol Connector:Conn_01x07_Socket
Connections:
- net GND: now also C41.1, J1.5 (Pin_5), J1.6 (Pin_6)
- net LED_FAULT: now also J1.1 (Pin_1); no longer J2.4 (Pin_4)
- net PWM_ADIM: now also J1.3 (Pin_3)
- net PWM_EN: now also J1.2 (Pin_2)
- net VCC: now also J2.4 (Pin_4), C41.2, J1.4 (Pin_4), J1.7 (Pin_7)
